Commit message: Added the lidar urdf and updated the rest

File: src/demo_bot/description/color_macro.xacro (robot description, xacro)
@@ -14,3 +14,6 @@
         <color rgba="0 0 0 1"/>
      </material>
+     <material name="red">
+      <color rgba="1 0 0 1"/>
+     </material>
 </robot>

File: src/demo_bot/description/robot.urdf.xacro (robot description, xacro)
@@ -3,3 +3,4 @@
     <xacro:include filename="robot_core.xacro"/>
     <xacro:include filename="ros2_control.xacro"/>
+    <xacro:include filename="lidar.xacro"/>
 </robot>
