Commit message: Moved it out front, haven't tested

File: src/demo_bot/description/depth_camera.xacro (robot description, xacro)
@@ -4,5 +4,5 @@
         <parent link="chassis"/>
         <child link='camera_link'/>
-        <origin xyz='0.305 0  0.08' rpy='0 0 0'/>
+        <origin xyz='0.305 0  0.1' rpy='0 0 0'/>
     </joint>
     <link name="camera_link">
@@ -28,5 +28,5 @@
             <pose>0 0 0 0 0 0</pose>
             <topic>camera</topic>
-            <gz_frame_id>camera_link</gz_frame_id>
+            <frame_id>camera_link</frame_id>
             <visualize>true</visualize>
             <update_rate>10</update_rate>
